Commit message: update

File: navcore_description/urdf/navcore.urdf (robot description, URDF)
Before this commit: robot navcore, 1 links, 0 joints
Links:
- link base_link: mass 35.336455 -> 1.0

Commit message: model

File: navcore_description/urdf/navcore.urdf (robot description, URDF)
Before this commit: robot navcore, 1 links, 0 joints
Links:
- added link wheel_l
- link base_link: mass 1.0 -> None; geometry 
